Commit message: modify the original pose

File: assets/mjcf/pliers/mobility.urdf (robot description, URDF)
Before this commit: robot partnet_2f4b18402dee61003f7c6295b60afd1b, 3 links, 2 joints
Links:
- link link_0: geometry collision mesh filename=textured_objs/original-2.obj scale=0.3 0.3 0.3; collision mesh filename=textured_objs/original-3.obj scale=0.3 0.3 0.3
- link link_1: geometry collision mesh filename=textured_objs/original-1.obj scale=0.3 0.3 0.3; collision mesh filename=textured_objs/original-4.obj scale=0.3 0.3 0.3
