Commit message: add glasses asset

File: assets/mjcf/toast.urdf (robot description, URDF)
Before this commit: robot box, 1 links, 0 joints
Links:
- link box: geometry collision box size=0.04 0.04 0.04; visual box size=0.2 0.2 0.05

File: assets/mjcf/toaster/mobility.urdf (robot description, URDF)
Before this commit: robot partnet_3ffbb0ab0f8da32f86271197b958e3d5, 4 links, 3 joints
Links:
- link link_0: geometry collision mesh filename=textured_objs/original-34.obj scale=0.3 0.3 0.3; visual mesh filename=textured_objs/original-34.obj scale=0.3 0.3 0.3
- link link_1: geometry collision mesh filename=textured_objs/original-33.obj scale=0.3 0.3 0.3; visual mesh filename=textured_objs/original-33.obj scale=0.3 0.3 0.3
- link link_2: geometry collision mesh filename=textured_objs/original-1.obj scale=0.3 0.3 0.3; collision mesh filename=textured_objs/original-10.obj scale=0.3 0.3 0.3

File: assets/urdf/ycb/061_foam_brick/061_foam_brick.urdf (robot description, URDF)
Before this commit: robot foam_brick, 1 links, 0 joints
Links:
- link foam_brick: geometry collision box size=0.049 0.074 0.049; visual mesh filename=ycb/061_foam_brick/textured.obj scale=0.04 0.04 0.04
